File: Z80computer_GC.kicad_sch (KiCad schematic)
At the start: 127 parts, among them J1 Conn_01x10_Pin, J2 Conn_01x10_Pin, M0 LED, SW1 SW_DIP_x01, SW7 SW_Slide_DPDT, U0 74HCT244, U1 74HCT244, U10 74HCT244, U11 74HCT244, U13 NE555P, U2 74HCT244, U3 74HCT244, U4 Z80CPU, U6 CY7C199, U8 74HCT244, U9 74HCT244, Y0 CXO_DIP8

Commit message: update
Connections:
- net A10: now also RN2.4 (R3), U1.6 (1A2)
- net A11: now also RN2.5 (R4), U1.8 (1A3)
- net A12: now also RN2.6 (R5), U1.17 (2A0)
- net A13: now also RN2.7 (R6), U1.15 (2A1)
- net A14: now also RN2.8 (R7), U1.13 (2A2)
- net A8: now also RN2.2 (R1), U1.2 (1A0)
- net A9: now also RN2.3 (R2), U1.4 (1A1)
- net GND: now also R31.2
- net VCC: no longer R31.1
- net PULL_DOWN: now reaches U0.1 (1OE), U0.19 (2OE), U1.1 (1OE), U1.19 (2OE), U2.1 (1OE), U2.19 (2OE), U3.1 (1OE), U3.19 (2OE)
- net PULL_DOWN: now also R31.1; no longer R31.2
- net CLOCK: now reaches RN0.2 (R1), SW7.2 (B), U3.2 (1A0), U4.6 (~{CLK}), Z80PIO0.25 (CLK)
- net M1: now reaches RN0.3 (R2), U3.4 (1A1), U4.27 (~{M1}), Z80PIO0.37 (~{M1})
- net WAIT: now reaches R34.2, RN0.4 (R3), U3.6 (1A2), U4.17 (~{NMI}), U4.24 (~{WAIT})
- net INT: now reaches U4.16 (~{INT}), Z80PIO0.23 (~{INT})
Other:
- moved on the sheet: 74HCT244-7, A0, A1, A2, A3, A4, A5, A6, A7, BUSACK0, C1, C2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

Commit message: updaate
Parts:
- removed 74HCT244-7, U0, U1, U10, U11, U2, U3, U8, U9: 74HCT244, Package_DIP:DIP-20_W7.62mm_Socket, symbol 74xx:74HCT244
- removed A0, A1, A10, A11, A12, A13, A14, A2, A3, A4, A5, A6, A7, A8, A9, BUSACK0, CLK0, D0, D1, D2, D3, D4, D5, D6, D7, IORQ0, M0, MREQ0, O0, O1, O2, O3, O4, O5, O6, O7, RD0, WAIT0, WR0: LED, LED_THT:LED_D3.0mm, symbol Device:LED
- removed A0-A7, A8-A14, D0-D7, I0-I7: SW_DIP_x08, Package_DIP:DIP-16_W7.62mm_Socket, symbol Switch:SW_DIP_x08
- removed C2, C3: 0.01u, Capacitor_THT:CP_Radial_D5.0mm_P2.00mm, symbol Device:C
- removed J1, J2: Conn_01x10_Pin, Connector_PinHeader_2.54mm:PinHeader_1x10_P2.54mm_Vertical, symbol Connector:Conn_01x10_Pin
- removed R0, R1, R10, R11, R12, R13, R14, R15, R16, R17, R18, R19, R2, R20, R21, R22, R23, R24, R25, R26, R27, R28, R29, R3, R30, R36, R37, R38, R4, R40, R41, R42, R43, R44, R45, R46, R47, R48, R5, R6, R7, R8, R9: 4.7k, Resistor_THT:R_Axial_DIN0204_L3.6mm_D1.6mm_P7.62mm_Horizontal, symbol Device:R
- removed R35: 330, Resistor_THT:R_Axial_DIN0204_L3.6mm_D1.6mm_P7.62mm_Horizontal, symbol Device:R
- removed R39: 10k, Resistor_THT:R_Axial_DIN0204_L3.6mm_D1.6mm_P7.62mm_Horizontal, symbol Device:R
- removed RN0, RN1, RN2, RN3, RN4, RN5, RN7, RN8: 4.7k, Resistor_THT:R_Array_SIP9, symbol Device:R_Network08
- removed RV0: R_Potentiometer, Potentiometer_THT:Potentiometer_ACP_CA9-H5_Horizontal, symbol Device:R_Potentiometer
- removed SW7: SW_Slide_DPDT, Button_Switch_THT:SW_E-Switch_EG1271_SPDT, symbol Switch:SW_Slide_DPDT
- removed U13: NE555P, Package_DIP:DIP-8_W7.62mm_Socket, symbol Timer:NE555P
- removed WRITE0: SW_Push, Button_Switch_THT:SW_PUSH_6mm, symbol Switch:SW_Push
- removed Y0: CXO_DIP8, Oscillator:Oscillator_DIP-8, symbol Oscillator:CXO_DIP8
- removed Z80PIO0: Z8420, Package_DIP:DIP-40_W15.24mm_Socket, symbol Interface:Z8420
Connections:
- no-connect marks 27 -> 3
Other:
- added sheet clock_generater (clock_generater.kicad_sch)
- added sheet data_address_debug_indicater (indicater.kicad_sch)
- added sheet data_address_input (input.kicad_sch)
- added sheet graphic_card (graphic_card.kicad_sch)
- added sheet input_output (input_output.kicad_sch)
- moved on the sheet: C0, C1, R31, R32, R33, R34, RESET0, SW1, TP0, TP1, U4, U6
