File: graphic_card.kicad_sch (KiCad schematic)
At the start: 0 parts

Commit message: started designing board
Parts:
- added U1, U2, U3: 74LS161, symbol 74xx:74LS161
- added Y1: CXO_DIP8, Oscillator:Oscillator_DIP-8, symbol Oscillator:CXO_DIP8
Connections:
- new net: U1.15 (TC), U2.10 (CET)
- new net: U2.15 (TC), U3.10 (CET)
- new net C0: U1.3 (D0)
- new net C1: U1.4 (D1)
- new net C10: U3.5 (D2)
- new net C11: U3.6 (D3)
- new net C2: U1.5 (D2)
- new net C3: U1.6 (D3)
- new net C4: U2.3 (D0)
- new net C5: U2.4 (D1)
- new net C6: U2.5 (D2)
- new net C7: U2.6 (D3)
- new net C8: U3.3 (D0)
- new net C9: U3.4 (D1)
- new net CLEAR: U1.1 (~{MR}), U2.1 (~{MR}), U3.1 (~{MR})
- new net CLOCK: U1.2 (CP), U2.2 (CP), U3.2 (CP), Y1.5 (OUT)
- new net GND: U1.8 (GND), U2.8 (GND), U3.8 (GND), Y1.4 (GND)
- new net VCC: U1.10 (CET), U1.16 (VCC), U1.7 (CEP), U1.9 (~{PE}), U2.16 (VCC), U2.7 (CEP), U2.9 (~{PE}), U3.16 (VCC), U3.7 (CEP), U3.9 (~{PE}), Y1.8 (Vcc)
- no-connect marks 0 -> 13
Other:
- added sheet timing_detector (timing_detector.kicad_sch)

Commit message: update
Connections:
- net C10: no longer names the net of U3.5 (D2)
- net C11: no longer names the net of U3.6 (D3)
- net C9: no longer names the net of U3.4 (D1)
- no-connect marks 13 -> 17
Changed lines of the file:
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@@
+	)
+	(no_connect
+		(at 123.19 158.75)
 	)
 	(no_connect
@@
 	)
 	(no_connect
+		(at 123.19 153.67)
+	)
+	(no_connect
 		(at 148.59 102.87)
 	)
 	(no_connect
+		(at 123.19 156.21)
+	)
+	(no_connect
 		(at 148.59 153.67)
 	)
@@
 	)
 	(no_connect
+		(at 148.59 163.83)
+	)
+	(no_connect
 		(at 148.59 151.13)
 	)
@@
 	)
 	(bus_entry
-		(at 118.11 153.67)
-		(size 2.54 2.54)
-		(stroke
-			(width 0)
-			(type default)
-		)
-	)
-	(bus_entry
 		(at 118.11 39.37)
 		(size 2.54 2.54)
@@
 	)
 	(bus_entry
-		(at 118.11 156.21)
-		(size 2.54 2.54)
-		(stroke
-			(width 0)
-			(type default)
-		)
-	)
-	(bus_entry
 		(at 118.11 92.71)
 		(size 2.54 2.54)
@@
 		)
 	)
-	(bus_entry
-		(at 118.11 151.13)
-		(size 2.54 2.54)
-		(stroke
-			(width 0)
-			(type default)
-		)
-	)
 	(wire
 		(pts
@@
 		)
 	)
-	(wire
-		(pts
-			(xy 120.65 156.21) (xy 123.19 156.21)
-		)
-		(stroke
-			(width 0)
-			(type default)
-		)
-	)
 	(bus
 		(pts
@@
 		)
 	)
-	(bus
-		(pts
-			(xy 118.11 151.13) (xy 118.11 153.67)
-		)
-		(stroke
-			(width 0)
-			(type default)
-		)
-	)
 	(wire
 		(pts
@@
 		)
 	)
-	(bus
-		(pts
-			(xy 118.11 148.59) (xy 118.11 151.13)
-		)
-		(stroke
-			(width 0)
-			(type default)
-		)
-	)
 	(wire
 		(pts
@@
 	(bus
 		(pts
-			(xy 118.11 153.67) (xy 118.11 156.21)
-		)
-		(stroke
-			(width 0)
-			(type default)
-		)
-	)
-	(bus
-		(pts
 			(xy 118.11 41.91) (xy 118.11 44.45)
 		)
@@
 	(wire
 		(pts
-			(xy 120.65 153.67) (xy 123.19 153.67)
-		)
-		(stroke
-			(width 0)
-			(type default)
-		)
-	)
-	(wire
-		(pts
 			(xy 101.6 163.83) (xy 123.19 163.83)
 		)
@@
 		(pts
 			(xy 114.3 168.91) (xy 123.19 168.91)
-		)
-		(stroke
-			(width 0)
-			(type default)
-		)
-	)
-	(wire
-		(pts
-			(xy 120.65 158.75) (xy 123.19 158.75)
 		)
 		(stroke
@@
 		)
 	)
-	(label "C10"
-		(at 121.92 156.21 0)
-		(effects
-			(font
-				(size 1.27 1.27)
-			)
-			(justify left bottom)
-		)
-	)
-	(label "C9"
-		(at 121.92 153.67 0)
-		(effects
-			(font
-				(size 1.27 1.27)
-			)
-			(justify left bottom)
-		)
-	)
 	(label "C2"
 		(at 121.92 44.45 0)
@@
 		(effects
 			(font
-				(size 1.27 1.27)
-			)
-			(justify left bottom)
-		)
-	)
-	(label "C11"
-		(at 121.92 158.75 0)
-		(effects
-			(font
