File: timing_detector.kicad_sch (KiCad schematic)
At the start: 1 part, among them U15 74LS30

Commit message: update
Parts:
- added U16, U17, U27, U28: 74LS04, symbol 74xx:74LS04
- added U18, U19, U20, U26: 74LS30, symbol 74xx:74LS30
- added U21: 74HC00, symbol 74xx:74HC00
Connections:
- net C0: now also U27.1
- net C1: now also U16.3, U18.2, U19.2
- net C2: now also U16.5, U20.3
- net C3: now also U15.4, U16.9
- net C4: now also U16.11, U18.5, U19.5
- net C5: now also U16.13, U19.6
- net C6: now also U15.11, U18.11, U19.11, U28.1
- net C7: now also U15.12, U17.3, U18.12, U19.12
- net C8: now also U17.5, U20.12
- net VCC: now reaches U15.14 (VCC)
- net VCC: now also U16.14 (VCC), U17.14 (VCC), U18.14 (VCC), U19.14 (VCC), U20.14 (VCC), U21.14 (VCC), U26.14 (VCC)
- net GND: now reaches U15.7 (GND)
- net GND: now also U16.7 (GND), U17.7 (GND), U18.7 (GND), U19.7 (GND), U20.7 (GND), U21.7 (GND), U26.7 (GND)
- net _C0: now reaches U15.1
- net _C0: now also U18.1, U19.1, U20.1, U27.2
- net _C1: now reaches U15.2
- net _C1: now also U16.4, U20.2
- net _C2: now reaches U15.3
- net _C2: now also U16.6, U18.3, U19.3
- net _C4: now reaches U15.5
- net _C4: now also U16.10, U20.5
- net _C5: now reaches U15.6
- net _C5: now also U16.12, U18.6, U20.6
- net _200: now reaches U15.8
- net _200: now also U21.5
- new net _210: U18.8, U21.9
- new net _242: U19.8, U21.13
- new net _264: U20.8, U21.1
- new net _C3: U16.8, U18.4, U19.4, U20.4
- new net _C6: U20.11, U28.2
- new net _C7: U17.4
- new net _C8: U17.6
- new net _display: U21.2, U21.6
- new net _h_sync: U21.12, U21.8
- new net display: U21.3, U21.4
- new net h_sync: U21.10, U21.11
- no-connect marks 0 -> 6
Other:
- moved on the sheet: U15A, U15B
